File: hardware/main_3_0.brd (EAGLE design)
At the start: 92.6 x 82.2 mm, 102 parts, among them IC1 24CL04BSM, IC2 LM2937, Q1 8MHz, Q2 BSS123, Q3 BSS123, U4 STM32F303RCT6, X1 MINI-USB-32005-201

Commit message: board
Parts:
- moved Q3 9.41 mm to (36.6, 15.2), flipped to the bottom
- moved R30 9.31 mm to (36.6, 18.1), flipped to the bottom
- moved R33 8.17 mm to (56.5, 14.2), turned to 180 degrees
- moved R32 0.86 mm to (52.0, 13.4), turned to 90 degrees
- moved LASER 0.73 mm to (80.1, 42.7)
- moved R14 0.41 mm to (37.3, 26.0)
Routing:
- net SDA: track 41.2 -> 158.7 mm, vias 1 -> 2
- net SCL: track 39.6 -> 154.0 mm, vias 3 -> 5
- net IR_LED_FRONT: track 143.6 -> 159.1 mm, vias 0 -> 1
- net IR_CONTROLL_FRONT: track 30.5 -> 15.2 mm, vias 2 -> 0
- net +3V3: track 408.0 -> 422.7 mm, vias 13 -> 14
- net N$24: track 3.11 -> 9.46 mm
- net ADC10: track 33.2 -> 39.1 mm
- net GND: track 633.1 -> 638.9 mm, vias 57 -> 54
- net BOOT: track 28.5 -> 33.8 mm
- net N$13: track 0.00 -> 3.58 mm
- net ADC9: track 43.8 -> 46.4 mm, vias 2 -> 3
Other:
- outline, holes or cut-outs redrawn

Commit message: board
Parts:
- added C17: 100n, resistor:C0805
- added C18: 10uF, resistor:C0805
- added LASER1: (no value), con-lstb:MA04-1
- added R35: 47k, resistor:M0805
- added U1: VL53L1XSMD, SparkFun-Sensors:VL53L1X
- moved Q3 4.34 mm to (40.8, 14.4), turned to 90 degrees
- moved R30 3.92 mm to (38.0, 14.4), turned to 270 degrees
- moved BOOT 2.80 mm to (41.8, 18.2), turned to 90 degrees
- moved IR_RIGHT 1.04 mm to (56.9, 75.2)
- moved IR_S_LEFT 0.41 mm to (51.0, 76.2)
Connections:
- net IR_CONTROLL renamed LINE_LED_CONTROLL
- new net LINE_LED: Q2.3
- new net N$26: C17.2, C18.2, LASER1.4, R35.2, U1.1, U1.11
- new net N$27: LASER1.1, U1.9
- new net N$28: LASER1.2, U1.10
- new net N$29: R35.1, U1.5
- net GND: now also C17.1, C18.1, LASER1.3, U1.12, U1.2, U1.3, U1.4, U1.6
- net IR_LED: no longer Q2.3
Routing:
- net GND: track 638.9 -> 663.3 mm, vias 54 -> 81
- net N$26: track 0.00 -> 20.9 mm, vias 0 -> 2
- net SDA: track 158.7 -> 176.7 mm, vias 2 -> 3
- net IR_CONTROLL_FRONT: track 15.2 -> 31.2 mm, vias 0 -> 1
- net SCL: track 154.0 -> 168.8 mm, vias 5 -> 6
- net IR_LED_FRONT: track 159.1 -> 151.8 mm
- net BOOT: track 33.8 -> 26.5 mm, vias 1 -> 2
- net N$27: track 0.00 -> 5.83 mm
- net N$28: track 0.00 -> 4.52 mm
- net +3V3: track 422.7 -> 419.3 mm
- net N$29: track 0.00 -> 2.53 mm, vias 0 -> 1
- net ADC9: track 46.4 -> 45.1 mm
- net N$24: track 9.46 -> 8.34 mm
- added copper zone on layer 1, net GND
- added copper zone on layer 16, net GND
Other:
- outline, holes or cut-outs redrawn
- board text added: "UART"
