File: hardware/main_3_0.sch (EAGLE design)
At the start: 102 parts, among them IC1 24CL04BSM, IC2 LM2937, Q1 8MHz, Q2 BSS123, Q3 BSS123, U4 STM32F303RCT6, X1 MINI-USB-32005-201

Commit message: board
Parts:
- added C17: 100n, resistor:C-EUC0805
- added C18: 10uF, resistor:C-EUC0805
- added LASER1: (no value), con-lstb:MA04-1
- added R35: 47k, resistor:R-EU_M0805
- added U1: VL53L1XSMD, SparkFun-Sensors:VL53L1XSMD
Connections:
- net IR_CONTROLL renamed LINE_LED_CONTROLL
- new net LINE_LED: Q2.D
- new net N$26: C17.2, C18.2, LASER1.4, R35.2, U1.VCC
- new net N$27: LASER1.1, U1.SDA
- new net N$28: LASER1.2, U1.SCL
- new net N$29: R35.1, U1.!SHUT
- net GND: now also C17.1, C18.1, LASER1.3, U1.GND
- net IR_LED: no longer Q2.D
Changed lines of the file:
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@@
 <layer number="59" name="tCarbon" color="7" fill="1" visible="no" active="no"/>
 <layer number="60" name="bCarbon" color="7" fill="1" visible="no" active="no"/>
+<layer number="88" name="SimResults" color="9" fill="1" visible="yes" active="yes"/>
+<layer number="89" name="SimProbes" color="9" fill="1" visible="yes" active="yes"/>
 <layer number="90" name="Modules" color="7" fill="1" visible="yes" active="yes"/>
 <layer number="91" name="Nets" color="2" fill="1" visible="yes" active="yes"/>
@@
 <layer number="112" name="tSilk" color="7" fill="1" visible="yes" active="yes"/>
 <layer number="113" name="ReferenceLS" color="7" fill="1" visible="yes" active="yes"/>
+<layer number="114" name="Badge_Outline" color="7" fill="1" visible="yes" active="yes"/>
+<layer number="115" name="ReferenceISLANDS" color="7" fill="1" visible="yes" active="yes"/>
 <layer number="116" name="Patch_BOT" color="9" fill="4" visible="yes" active="yes"/>
 <layer number="118" name="Rect_Pads" color="7" fill="1" visible="yes" active="yes"/>
@@
 <part name="GND60" library="supply1" deviceset="GND" device=""/>
 <part name="+3V45" library="supply1" deviceset="+3V3" device=""/>
+<part name="U1" library="SparkFun-Sensors" deviceset="VL53L1X" device="SMD"/>
+<part name="LASER1" library="con-lstb" deviceset="MA04-1" device=""/>
+<part name="R35" library="resistor" deviceset="R-EU_" device="M0805" value="47k"/>
+<part name="C17" library="resistor" deviceset="C-EU" device="C0805" value="100n"/>
+<part name="C18" library="resistor" deviceset="C-EU" device="C0805" value="10uF"/>
+<part name="GND61" library="supply1" deviceset="GND" device=""/>
 </parts>
 <sheets>
@@
 <instance part="GND60" gate="1" x="469.9" y="77.47" rot="R270"/>
 <instance part="+3V45" gate="G$1" x="474.98" y="69.85" rot="R180"/>
+<instance part="U1" gate="U1" x="547.37" y="80.01"/>
+<instance part="LASER1" gate="1" x="499.11" y="77.47" rot="MR180"/>
+<instance part="R35" gate="G$1" x="552.45" y="95.25" rot="R180"/>
+<instance part="C17" gate="G$1" x="523.24" y="80.01" rot="R180"/>
+<instance part="C18" gate="G$1" x="530.86" y="80.01" rot="R180"/>
+<instance part="GND61" gate="1" x="527.05" y="71.12"/>
 </instances>
 <busses>
@@
 <pinref part="GND60" gate="1" pin="GND"/>
 </segment>
+<segment>
+<pinref part="U1" gate="U1" pin="GND"/>
+<pinref part="LASER1" gate="1" pin="3"/>
+<wire x1="537.21" y1="77.47" x2="530.86" y2="77.47" width="0.1524" layer="91"/>
+<pinref part="C17" gate="G$1" pin="1"/>
+<wire x1="530.86" y1="77.47" x2="527.05" y2="77.47" width="0.1524" layer="91"/>
+<wire x1="527.05" y1="77.47" x2="523.24" y2="77.47" width="0.1524" layer="91"/>
+<wire x1="523.24" y1="77.47" x2="506.73" y2="77.47" width="0.1524" layer="91"/>
+<junction x="523.24" y="77.47"/>
+<pinref part="C18" gate="G$1" pin="1"/>
+<junction x="530.86" y="77.47"/>
+<pinref part="GND61" gate="1" pin="GND"/>
+<wire x1="527.05" y1="73.66" x2="527.05" y2="77.47" width="0.1524" layer="91"/>
+<junction x="527.05" y="77.47"/>
+</segment>
 </net>
 <net name="VCC" class="0">
@@
 <wire x1="241.3" y1="111.76" x2="228.6" y2="111.76" width="0.1524" layer="91"/>
 <label x="226.06" y="111.76" size="1.778" layer="95" rot="R180"/>
-</segment>
-</net>
-<net name="IR_CONTROLL" class="0">
-<segment>
-<pinref part="U4" gate="B" pin="PA8"/>
-<wire x1="276.86" y1="106.68" x2="284.48" y2="106.68" width="0.1524" layer="91"/>
-<label x="289.56" y="106.68" size="1.778" layer="95"/>
-</segment>
-<segment>
-<pinref part="Q2" gate="G$1" pin="G"/>
-<pinref part="R3" gate="G$1" pin="2"/>
-<wire x1="30.48" y1="121.92" x2="27.94" y2="121.92" width="0.1524" layer="91"/>
-<wire x1="27.94" y1="121.92" x2="27.94" y2="116.84" width="0.1524" layer="91"/>
-<wire x1="27.94" y1="121.92" x2="17.78" y2="121.92" width="0.1524" layer="91"/>
-<junction x="27.94" y="121.92"/>
-<label x="12.7" y="124.46" size="1.778" layer="95"/>
 </segment>
 </net>
@@
 <label x="243.84" y="162.56" size="1.778" layer="95" rot="R270"/>
 </segment>
-<segment>
-<pinref part="Q2" gate="G$1" pin="D"/>
-<wire x1="35.56" y1="129.54" x2="35.56" y2="134.62" width="0.1524" layer="91"/>
-<label x="40.64" y="134.62" size="1.778" layer="95"/>
-</segment>
 </net>
 <net name="N$15" class="0">
@@
 </segment>
 </net>
+<net name="LINE_LED" class="0">
+<segment>
+<pinref part="Q2" gate="G$1" pin="D"/>
+<wire x1="35.56" y1="129.54" x2="35.56" y2="134.62" width="0.1524" layer="91"/>
+<label x="40.64" y="134.62" size="1.778" layer="95"/>
+</segment>
+</net>
+<net name="LINE_LED_CONTROLL" class="0">
+<segment>
+<pinref part="Q2" gate="G$1" pin="G"/>
+<pinref part="R3" gate="G$1" pin="2"/>
+<wire x1="30.48" y1="121.92" x2="27.94" y2="121.92" width="0.1524" layer="91"/>
+<wire x1="27.94" y1="121.92" x2="27.94" y2="116.84" width="0.1524" layer="91"/>
+<wire x1="27.94" y1="121.92" x2="17.78" y2="121.92" width="0.1524" layer="91"/>
+<junction x="27.94" y="121.92"/>
+<label x="12.7" y="124.46" size="1.778" layer="95"/>
+</segment>
+<segment>
+<pinref part="U4" gate="B" pin="PA8"/>
+<wire x1="276.86" y1="106.68" x2="284.48" y2="106.68" width="0.1524" layer="91"/>
+<label x="289.56" y="106.68" size="1.778" layer="95"/>
+</segment>
+</net>
+<net name="N$26" class="0">
+<segment>
+<pinref part="LASER1" gate="1" pin="4"/>
+<wire x1="506.73" y1="74.93" x2="515.62" y2="74.93" width="0.1524" layer="91"/>
+<wire x1="515.62" y1="74.93" x2="515.62" y2="85.09" width="0.1524" layer="91"/>
+<pinref part="U1" gate="U1" pin="VCC"/>
+<wire x1="515.62" y1="85.09" x2="523.24" y2="85.09" width="0.1524" layer="91"/>
+<pinref part="R35" gate="G$1" pin="2"/>
+<wire x1="523.24" y1="85.09" x2="530.86" y2="85.09" width="0.1524" layer="91"/>
+<wire x1="530.86" y1="85.09" x2="535.94" y2="85.09" width="0.1524" layer="91"/>
+<wire x1="535.94" y1="85.09" x2="537.21" y2="85.09" width="0.1524" layer="91"/>
+<wire x1="547.37" y1="95.25" x2="535.94" y2="95.25" width="0.1524" layer="91"/>
+<wire x1="535.94" y1="95.25" x2="535.94" y2="85.09" width="0.1524" layer="91"/>
+<junction x="535.94" y="85.09"/>
+<pinref part="C17" gate="G$1" pin="2"/>
+<junction x="523.24" y="85.09"/>
+<pinref part="C18" gate="G$1" pin="2"/>
+<junction x="530.86" y="85.09"/>
+</segment>
+</net>
+<net name="N$27" class="0">
+<segment>
+<pinref part="U1" gate="U1" pin="SDA"/>
+<wire x1="557.53" y1="82.55" x2="562.61" y2="82.55" width="0.1524" layer="91"/>
+<wire x1="562.61" y1="82.55" x2="562.61" y2="91.44" width="0.1524" layer="91"/>
+<wire x1="562.61" y1="91.44" x2="509.27" y2="91.44" width="0.1524" layer="91"/>
+<wire x1="509.27" y1="91.44" x2="509.27" y2="82.55" width="0.1524" layer="91"/>
+<pinref part="LASER1" gate="1" pin="1"/>
+<wire x1="509.27" y1="82.55" x2="506.73" y2="82.55" width="0.1524" layer="91"/>
+</segment>
+</net>
+<net name="N$28" class="0">
+<segment>
+<pinref part="U1" gate="U1" pin="SCL"/>
+<wire x1="557.53" y1="80.01" x2="561.34" y2="80.01" width="0.1524" layer="91"/>
+<wire x1="561.34" y1="80.01" x2="561.34" y2="90.17" width="0.1524" layer="91"/>
+<wire x1="561.34" y1="90.17" x2="510.54" y2="90.17" width="0.1524" layer="91"/>
+<wire x1="510.54" y1="90.17" x2="510.54" y2="80.01" width="0.1524" layer="91"/>
+<pinref part="LASER1" gate="1" pin="2"/>
+<wire x1="510.54" y1="80.01" x2="506.73" y2="80.01" width="0.1524" layer="91"/>
+</segment>
+</net>
+<net name="N$29" class="0">
+<segment>
+<pinref part="U1" gate="U1" pin="!SHUT"/>
+<wire x1="557.53" y1="85.09" x2="560.07" y2="85.09" width="0.1524" layer="91"/>
+<wire x1="560.07" y1="85.09" x2="560.07" y2="95.25" width="0.1524" layer="91"/>
+<pinref part="R35" gate="G$1" pin="1"/>
+<wire x1="560.07" y1="95.25" x2="557.53" y2="95.25" width="0.1524" layer="91"/>
+</segment>
+</net>
